File: 電子回路/raspberryPi/raspberryPi.kicad_sch (KiCad schematic)
At the start: 20 parts, among them J1 Conn_01x05_Pin, J10 Screw_Terminal_01x01, J2 Conn_01x04_Pin, J3 Conn_01x01_Pin, J4 Screw_Terminal_01x01, J5 Screw_Terminal_01x01, J6 Screw_Terminal_01x01, J7 Screw_Terminal_01x01, J8 Screw_Terminal_01x01, J9 Screw_Terminal_01x01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

Commit message: 電子回路修正_202310202310
Parts:
- removed C1: C_Polarized_Small, symbol Device:C_Polarized_Small
- removed Q1: NMOS, symbol Simulation_SPICE:NMOS
- added BT1: Battery_Cell, symbol Device:Battery_Cell
- added D2: D, symbol Device:D
- added K6: Relay_SPST-NO, symbol Relay:Relay_SPST-NO
- added U1: 74HC86, symbol 74xx:74HC86
- added U2: MCP3002, symbol Analog_ADC:MCP3002
Connections:
- net +5V: now also D2.2 (A), U1.1; no longer D1.2 (A)
- net GND: now also BT1.2 (-)
- net power_IN: now also R1.1; no longer D1.1 (K)
- net systemStartPin: now reaches RP1.12 (GPIO_18/PWM0/SPI1_CS0)
- net systemStartPin: now also K6.A2
- net at RP1.23 (GPIO_11/SPI0_SCLK): now also U2.7 (CLK)
- new net: D2.1 (K), U2.2 (CH0)
